File: STM32F745VE_Hardware/REV1.1/STM32F745VE_REV1.1.kicad_pcb (KiCad board)
At the start: 4 copper layers, 50 x 50 mm, 66 parts, among them J1 CONNECTOR_RJ45_SI-60062, J2 SOCKET_MICRO_SD_SMT_3M, J3 USB_MINI_B_SMD, J4 USB_MINI_B_SMD, P1 CONN_1x4, P2 Header_2x17, P3 Header_2x17, P4 Header_2x1, P5 Header_2x1, SW1 PUSHBUTTON_SPST_6MM_SMD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

Commit message: Rev 1.1 update
Parts:
- moved C16 6.39 mm to (62.0, 141.8), turned to 270 degrees
- moved C21 4.15 mm to (60.2, 141.8)
- moved P4 2.03 mm to (74.2, 144.0)
- moved R8 1.76 mm to (57.1, 129.0), turned to 0 degrees
- moved C17 1.16 mm to (75.9, 135.5), turned to 45 degrees
- moved C22 1.08 mm to (77.0, 136.6), turned to 45 degrees
- moved J2 0.72 mm to (58.5, 146.8)
- moved C25 0.71 mm to (57.1, 127.4), turned to 180 degrees
Routing:
- net /SDMMC_D0: track 34.6 -> 79.4 mm
- net /ETH_MDIO: track 38.1 -> 77.1 mm, vias 4 -> 6
- net /ETH_REF_CLK: track 7.69 -> 41.5 mm
- net /SDMMC_D2: track 60.6 -> 27.8 mm
- net /GPIO_20: track 42.0 -> 72.6 mm, vias 1 -> 2
- net /DAC_0: track 43.1 -> 15.3 mm, vias 2 -> 0
- net /I2C1_SCL: track 52.2 -> 27.3 mm, vias 3 -> 0
- net /USB_FS_DM: track 37.8 -> 16.1 mm, vias 0 -> 2
- net Net-(C6-Pad1): track 27.9 -> 6.89 mm, vias 3 -> 1
- net /GPIO_18: track 24.6 -> 42.2 mm, vias 1 -> 0
- net /MCU_RST: track 99.8 -> 83.3 mm, vias 6 -> 3
- net /I2C4_SCL: track 38.1 -> 24.3 mm
- net /USB_HS_DP: track 13.1 -> 25.6 mm, vias 0 -> 2
- net /VBATT: track 77.0 -> 64.6 mm, vias 2 -> 1
- net /GPIO_4: track 20.2 -> 31.7 mm
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