File: STM32F745VE_Hardware/REV1.1/preroute.kicad_pcb (KiCad board)
At the start: 4 copper layers, 50 x 50 mm, 66 parts, among them J1 CONNECTOR_RJ45_SI-60062, J2 SOCKET_MICRO_SD_SMT_3M, J3 USB_MINI_B_SMD, J4 USB_MINI_B_SMD, P1 CONN_1x4, P2 Header_2x17, P3 Header_2x17, P4 Header_2x1, P5 Header_2x1, SW1 PUSHBUTTON_SPST_6MM_SMD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

Commit message: Rev 1.1 update
Parts:
- moved P4 3.63 mm to (73.8, 141.2), turned to 180 degrees
- moved R8 1.76 mm to (57.1, 129.0), turned to 0 degrees
- moved J2 0.72 mm to (58.5, 146.8)
- moved C25 0.71 mm to (57.1, 127.4), turned to 180 degrees
Routing:
- net /+3.3VEXT: track 49.4 -> 0.00 mm
- net GND: track 47.6 -> 0.00 mm, vias 10 -> 0
- net +3.3V: track 46.1 -> 0.00 mm, vias 7 -> 0
- net /ETH_RXM: track 24.7 -> 0.00 mm
- net /ETH_RXP: track 20.6 -> 0.00 mm
- net /ETH_TXM: track 15.1 -> 0.00 mm
- net /OSCHSIN: track 14.4 -> 0.00 mm, vias 1 -> 0
- net /+3.0VREF: track 9.44 -> 0.00 mm
- net /ETH_TXP: track 9.20 -> 0.00 mm
- net /OSCHSOUT: track 9.18 -> 0.00 mm, vias 1 -> 0
- net /OSC32OUT: track 8.71 -> 0.00 mm
- net /OSC32IN: track 8.36 -> 0.00 mm
- net /+3.3VANA: track 7.57 -> 0.00 mm
- net /VCAP1: track 6.36 -> 0.00 mm, vias 1 -> 0
- net Net-(D1-Pad6): track 5.19 -> 0.00 mm
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Other:
- net class Default: via_dia 0.8128 -> 0.6096; via_drill 0.4064 -> 0.2032
- net class HI_POWER added: clearance 0.1778, trace_width 0.381, via_dia 0.8128, via_drill 0.4064
- rule via_min_drill: 0.254 -> 0.2032
